Commit message: Add arm link to simple robot model

File: ros2_ws/install/arm_lab/share/arm_lab/urdf/simple_robot.urdf.xacro (robot description, xacro)
@@ -3,30 +3,37 @@
        xmlns:xacro="http://www.ros.org/wiki/xacro">
   <xacro:property name="camera_height" value="1.0"/>
-  <link name="base_link">
-    <visual>
-      <geometry>
-        <box size="0.5 0.3 0.1"/>
-      </geometry>
-      <material name="blue">
-        <color rgba="0 0 1 1"/>
-      </material>
-    </visual>
-  </link>
-  <link name="camera_link">
-    <visual>
-      <geometry>
-        <box size="0.1 0.1 0.1"/>
-      </geometry>
-      <material name="red">
-        <color rgba="1 0 0 1"/>
-      </material>
-    </visual>
-  </link>
+  <xacro:macro name="box_link" params="name size color">
+    <link name="${name}">
+      <visual>
+        <geometry>
+          <box size="${size}"/>
+        </geometry>
+        <material name="${name}_material">
+          <color rgba="${color}"/>
+        </material>
+      </visual>
+    </link>
+  </xacro:macro>
+  <xacro:box_link
+    name="base_link"
+    size="0.5 0.3 0.1"
+    color="0 0 1 1"/>
+  <xacro:box_link
+    name="arm_link"
+    size="0.1 0.1 0.6"
+    color="0 1 0 1"/>
+  <xacro:box_link
+    name="camera_link"
+    size="0.1 0.1 0.1"
+    color="1 0 0 1"/>
+  <joint name="base_to_arm_joint" type="fixed">
+  <parent link="base_link"/>
+  <child link="arm_link"/>
+  <origin xyz="0 0 0.35" rpy="0 0 0"/>
+  </joint>
   <joint name="base_to_camera_joint" type="fixed">
-    <parent link="base_link"/>
+    <parent link="arm_link"/>
     <child link="camera_link"/>
-    <origin
-      xyz="0 0 ${camera_height}"
-      rpy="0 0 0"/>
+    <origin xyz="0 0 0.4" rpy="0 0 0"/>
   </joint>
 </robot>

Commit message: Add 2-DOF arm model with joint visualization

File: ros2_ws/install/arm_lab/share/arm_lab/urdf/simple_robot.urdf.xacro (robot description, xacro)
@@ -20,18 +20,34 @@
     color="0 0 1 1"/>
   <xacro:box_link
-    name="arm_link"
+    name="arm_link_1"
     size="0.1 0.1 0.6"
     color="0 1 0 1"/>
+  <xacro:box_link
+    name="arm_link_2"
+    size="0.1 0.1 0.5"
+    color="1 1 0 1"/>
   <xacro:box_link
     name="camera_link"
     size="0.1 0.1 0.1"
     color="1 0 0 1"/>
-  <joint name="base_to_arm_joint" type="fixed">
-  <parent link="base_link"/>
-  <child link="arm_link"/>
-  <origin xyz="0 0 0.35" rpy="0 0 0"/>
+  <joint name="base_to_arm_joint" type="revolute">
+    <parent link="base_link"/>
+    <child link="arm_link_1"/>
+    <origin xyz="0 0 0.35" rpy="0 0 0"/>
+    <axis xyz="0 0 1"/>
+    <limit lower="-1.57" upper="1.57" effort="10" velocity="1.0"/>
+  </joint>
+  <joint name="arm1_to_arm2_joint" type="revolute">
+    <parent link="arm_link_1"/>
+    <child link="arm_link_2"/>
+    <origin xyz="0 0 0.55" rpy="0 0 0"/>
+    <axis xyz="0 1 0"/>
+    <limit lower="-1.57"
+         upper="1.57"
+         effort="10"
+         velocity="1.0"/>
   </joint>
   <joint name="base_to_camera_joint" type="fixed">
-    <parent link="arm_link"/>
+    <parent link="arm_link_2"/>
     <child link="camera_link"/>
     <origin xyz="0 0 0.4" rpy="0 0 0"/>

Commit message: Add collision and inertial properties to robot links

File: ros2_ws/install/arm_lab/share/arm_lab/urdf/simple_robot.urdf.xacro (robot description, xacro)
@@ -13,4 +13,16 @@
         </material>
       </visual>
+      <collision>
+  	<geometry>
+    	  <box size="${size}"/>
+  	</geometry>
+      </collision>
+      <inertial>
+        <mass value="1.0"/>
+          <inertia
+    	     ixx="0.01" ixy="0.0" ixz="0.0"
+    	     iyy="0.01" iyz="0.0"
+             izz="0.01"/>
+      </inertial>
     </link>
   </xacro:macro>
@@ -48,5 +60,5 @@
          velocity="1.0"/>
   </joint>
-  <joint name="base_to_camera_joint" type="fixed">
+  <joint name="arm2_to_camera_joint" type="fixed">
     <parent link="arm_link_2"/>
     <child link="camera_link"/>

Commit message: Add Docker environment for ROS 2 Humble

File: ros2_ws/install/arm_lab/share/arm_lab/urdf/simple_robot.urdf.xacro (robot description, xacro)
@@ -65,3 +65,25 @@
     <origin xyz="0 0 0.4" rpy="0 0 0"/>
   </joint>
+  <ros2_control name="GazeboSystem" type="system">
+  <hardware>
+    <plugin>gz_ros2_control/GazeboSimSystem</plugin>
+  </hardware>
+  <joint name="base_to_arm_joint">
+    <command_interface name="position"/>
+    <state_interface name="position"/>
+    <state_interface name="velocity"/>
+  </joint>
+  <joint name="arm1_to_arm2_joint">
+    <command_interface name="position"/>
+    <state_interface name="position"/>
+    <state_interface name="velocity"/>
+  </joint>
+</ros2_control>
+<gazebo>
+  <plugin
+    filename="gz_ros2_control-system"
+    name="gz_ros2_control::GazeboSimROS2ControlPlugin">
+    <parameters>/home/akasha/MoMa-ArmLab/ros2_ws/install/arm_lab/share/arm_lab/config/arm_controllers.yaml</parameters>
+  </plugin>
+</gazebo>
 </robot>

Commit message: Add MoveIt configuration for 2-DOF arm

File: ros2_ws/install/arm_lab/share/arm_lab/urdf/simple_robot.urdf.xacro (robot description, xacro)
@@ -43,4 +43,8 @@
     size="0.1 0.1 0.1"
     color="1 0 0 1"/>
+  <xacro:box_link
+    name="tool0"
+    size="0.05 0.05 0.05"
+    color="1 0 1 1"/>
   <joint name="base_to_arm_joint" type="revolute">
     <parent link="base_link"/>
@@ -64,4 +68,9 @@
     <child link="camera_link"/>
     <origin xyz="0 0 0.4" rpy="0 0 0"/>
+  </joint>
+  <joint name="arm2_to_tool0_joint" type="fixed">
+    <parent link="arm_link_2"/>
+    <child link="tool0"/>
+    <origin xyz="0 0 0.3" rpy="0 0 0"/>
   </joint>
   <ros2_control name="GazeboSystem" type="system">
